File: I2C-GPIO.kicad_sch (KiCad schematic)
At the start: 1 part, among them U409 TCA9535DBR

Commit message: layout go brrr
Parts:
- added C439: 100nF, PCM_JLCPCB:C_0402, symbol PCM_JLCPCB-Capacitors:0402,100nF,(2)
- added R450, R451, R452, R454, R455, R456: 10kΩ, PCM_JLCPCB:R_0402, symbol PCM_JLCPCB-Resistors:0402,10kΩ
Connections:
- net GND: now reaches U409.12 (GND)
- net GND: now also C439.2, R451.2, R454.2, R455.2
- net at U409.2 (A1): now also R452.2, R455.1
- net at U409.21 (A0): now also R454.1, R456.2
- net GPIO.SCL: now reaches U409.22 (SCL)
- net GPIO.SDA: now reaches U409.23 (SDA)
- net +5V: now reaches U409.24 (VCC)
- net +5V: now also C439.1, R450.1, R452.1, R456.1
- net at U409.3 (A2): now also R450.2, R451.1
- no-connect marks 0 -> 9
