File: Power_Switch.kicad_sch (KiCad schematic)
At the start: 14 parts, among them Q400 MMBT2222A, Q401 MMBT2222A, Q402 AO3401A, Q403 AO3401A, U401 SN74LVC1G19DBVR

Commit message: layout go brrr
Parts:
- renumbered D411 to D404, R414 to R408, R415 to R409, R416 to R413, R418 to R414, R419 to R415
Connections:
- net SEL renamed GPIO.SEL
- net ~{EN} renamed GPIO.EN
