File: Hbridge.kicad_sch (KiCad schematic)
At the start: 8 parts, among them U403 DRV8844PWPR

Commit message: layout go brrr
Parts:
- C407, C408: footprint (none) -> Capacitor_SMD:CP_Elec_10x10
Connections:
- net EN1 is gone; now on net BRIDGE.EN1: U403.26 (EN1)
- net EN2 is gone; now on net BRIDGE.EN2: U403.24 (EN2)
- net EN3 is gone; now on net BRIDGE.EN3: U403.22 (EN3)
- net EN4 is gone; now on net BRIDGE.EN4: U403.20 (EN4)
- net IN1 is gone; now on net BRIDGE.IN1: U403.27 (IN1)
- net IN2 is gone; now on net BRIDGE.IN2: U403.25 (IN2)
- net IN3 is gone; now on net BRIDGE.IN3: U403.23 (IN3)
- net IN4 is gone; now on net BRIDGE.IN4: U403.21 (IN4)
- net NFAULT1 is gone; now on net BRIDGE.NFAULT: U403.18 (NFAULT)
- net NRST1 is gone; now on net BRIDGE.NRST: U403.16 (NRESET)
- net NSLEEP1 is gone; now on net BRIDGE.NSLEEP: U403.17 (NSLEEP)
Changed lines of the file:
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@@
+	)
+	(junction
+		(at 73.66 74.93)
+		(diameter 0)
+		(color 0 0 0 0)
 	)
 	(junction
@@
 		(color 0 0 0 0)
 	)
+	(junction
+		(at 59.69 92.71)
+		(diameter 0)
+		(color 0 0 0 0)
+	)
 	(no_connect
 		(at 128.27 95.25)
@@
 	(wire
 		(pts
+			(xy 172.72 113.03) (xy 172.72 110.49)
+		)
+		(stroke
+			(width 0)
+			(type default)
+		)
+	)
+	(wire
+		(pts
 			(xy 172.72 102.87) (xy 172.72 100.33)
 		)
@@
 	(wire
 		(pts
+			(xy 59.69 92.71) (xy 73.66 92.71)
+		)
+		(stroke
+			(width 0)
+			(type default)
+		)
+	)
+	(wire
+		(pts
 			(xy 104.14 80.01) (xy 128.27 80.01)
 		)
@@
 	(wire
 		(pts
-			(xy 57.15 92.71) (xy 73.66 92.71)
-		)
-		(stroke
-			(width 0)
-			(type default)
-		)
-	)
-	(wire
-		(pts
-			(xy 106.68 109.22) (xy 106.68 100.33)
+			(xy 45.72 92.71) (xy 59.69 92.71)
+		)
+		(stroke
+			(width 0)
+			(type default)
+		)
+	)
+	(wire
+		(pts
+			(xy 59.69 74.93) (xy 59.69 92.71)
+		)
+		(stroke
+			(width 0)
+			(type default)
+		)
+	)
+	(wire
+		(pts
+			(xy 106.68 111.76) (xy 106.68 100.33)
 		)
 		(stroke
@@
 		)
 	)
+	(wire
+		(pts
+			(xy 73.66 74.93) (xy 59.69 74.93)
+		)
+		(stroke
+			(width 0)
+			(type default)
+		)
+	)
 	(bus
 		(pts
@@
 			(width 0)
 			(type default)
+		)
+	)
+	(label "BRIDGE.NSLEEP"
+		(at 176.53 95.25 0)
+		(effects
+			(font
+				(size 1.27 1.27)
+			)
+			(justify left bottom)
 		)
 	)
@@
 		)
 	)
+	(label "BRIDGE.NRST"
+		(at 176.53 97.79 0)
+		(effects
+			(font
+				(size 1.27 1.27)
+			)
+			(justify left bottom)
+		)
+	)
+	(label "BRIDGE.EN1"
+		(at 176.53 72.39 0)
+		(effects
+			(font
+				(size 1.27 1.27)
+			)
+			(justify left bottom)
+		)
+	)
 	(label "GPIO1.Bridge+"
 		(at 111.76 85.09 0)
@@
 		)
 	)
+	(label "BRIDGE.EN2"
+		(at 176.53 77.47 0)
+		(effects
+			(font
+				(size 1.27 1.27)
+			)
+			(justify left bottom)
+		)
+	)
 	(label "BRIDGE.NRST"
 		(at 217.17 102.87 0)
@@
 		)
 	)
-	(label "IN3"
-		(at 176.53 80.01 0)
-		(effects
-			(font
-				(size 1.27 1.27)
-			)
-			(justify left bottom)
-		)
-	)
 	(label "GPIO1.Bridge-"
 		(at 210.82 121.92 0)
@@
 		)
 	)
-	(label "IN1"
-		(at 176.53 69.85 0)
-		(effects
-			(font
-				(size 1.27 1.27)
-			)
-			(justify left bottom)
-		)
-	)
 	(label "BRIDGE.IN2"
 		(at 217.17 80.01 0)
@@
 		)
 	)
-	(label "IN2"
-		(at 176.53 74.93 0)
+	(label "BRIDGE.EN3"
+		(at 176.53 82.55 0)
 		(effects
 			(font
@@
 		)
 	)
-	(label "IN4"
-		(at 176.53 85.09 0)
-		(effects
-			(font
-				(size 1.27 1.27)
-			)
-			(justify left bottom)
-		)
-	)
-	(label "NRST1"
-		(at 176.53 97.79 0)
-		(effects
-			(font
-				(size 1.27 1.27)
-			)
-			(justify left bottom)
-		)
-	)
-	(label "EN1"
-		(at 176.53 72.39 0)
-		(effects
-			(font
-				(size 1.27 1.27)
-			)
-			(justify left bottom)
-		)
-	)
-	(label "EN2"
-		(at 176.53 77.47 0)
-		(effects
-			(font
-				(size 1.27 1.27)
-			)
-			(justify left bottom)
-		)
-	)
 	(label "GPIO2.Bridge+"
 		(at 210.82 133.35 0)
@@
 		)
 	)
+	(label "BRIDGE.IN3"
+		(at 176.53 80.01 0)
+		(effects
+			(font
+				(size 1.27 1.27)
+			)
+			(justify left bottom)
+		)
+	)
 	(label "BRIDGE.IN4"
 		(at 217.17 85.09 0)
@@
 		)
 	)
-	(label "NSLEEP1"
-		(at 176.53 95.25 0)
+	(label "BRIDGE.EN4"
+		(at 176.53 87.63 0)
+		(effects
+			(font
+				(size 1.27 1.27)
+			)
+			(justify left bottom)
+		)
+	)
+	(label "BRIDGE.IN4"
+		(at 176.53 85.09 0)
 		(effects
 			(font
@@
 		)
 	)
-	(label "EN4"
-		(at 176.53 87.63 0)
-		(effects
-			(font
-				(size 1.27 1.27)
-			)
-			(justify left bottom)
-		)
-	)
-	(label "EN3"
-		(at 176.53 82.55 0)
+	(label "BRIDGE.NFAULT"
+		(at 176.53 92.71 0)
+		(effects
+			(font
+				(size 1.27 1.27)
+			)
+			(justify left bottom)
+		)
+	)
+	(label "BRIDGE.IN2"
+		(at 176.53 74.93 0)
 		(effects
 			(font
@@
 		)
 	)
+	(label "BRIDGE.IN1"
+		(at 176.53 69.85 0)
+		(effects
+			(font
+				(size 1.27 1.27)
+			)
+			(justify left bottom)
+		)
+	)
 	(label "BRIDGE.NFAULT"
 		(at 217.17 97.79 0)
@@
 		)
 	)
-	(label "NFAULT1"
-		(at 176.53 92.71 0)
-		(effects
-			(font
-				(size 1.27 1.27)
-			)
-			(justify left bottom)
-		)
-	)
 	(hierarchical_label "V_conn"
 		(shape input)
-		(at 57.15 92.71 180)
+		(at 45.72 92.71 180)
 		(effects
 			(font
@@
 			)
 		)
-		(property "Footprint" ""
+		(property "Footprint" "Capacitor_SMD:CP_Elec_10x10"
 			(at 74.6252 102.87 0)
 			(effects
@@
 	(symbol
 		(lib_id "power:GND")
-		(at 172.72 110.49 0)
+		(at 172.72 113.03 0)
 		(mirror y)
 		(unit 1)
@@
 		(fields_autoplaced yes)
 		(property "Reference" "#PWR0486"
-			(at 172.72 116.84 0)
+			(at 172.72 119.38 0)
 			(effects
 				(font
@@
 		)
 		(property "Value" "GND"
-			(at 172.72 115.57 0)
+			(at 172.72 118.11 0)
 			(effects
 				(font
@@
 		)
 		(property "Footprint" ""
-			(at 172.72 110.49 0)
+			(at 172.72 113.03 0)
 			(effects
 				(font
@@
 		)
 		(property "Datasheet" ""
-			(at 172.72 110.49 0)
+			(at 172.72 113.03 0)
 			(effects
 				(font
@@
 		)
 		(property "Description" "Power symbol creates a global label with name \"GND\" , ground"
-			(at 172.72 110.49 0)
+			(at 172.72 113.03 0)
 			(effects
 				(font
@@
 	(symbol
 		(lib_id "power:GND")
-		(at 106.68 109.22 0)
+		(at 106.68 111.76 0)
 		(mirror y)
 		(unit 1)
@@
 		(fields_autoplaced yes)
 		(property "Reference" "#PWR0482"
-			(at 106.68 115.57 0)
+			(at 106.68 118.11 0)
 			(effects
 				(font
@@
 		)
 		(property "Value" "GND"
-			(at 106.68 114.3 0)
+			(at 106.68 116.84 0)
 			(effects
 				(font
@@
 		)
 		(property "Footprint" ""
-			(at 106.68 109.22 0)
+			(at 106.68 111.76 0)
 			(effects
 				(font
@@
 		)
 		(property "Datasheet" ""
-			(at 106.68 109.22 0)
+			(at 106.68 111.76 0)
 			(effects
 				(font
@@
 		)
 		(property "Description" "Power symbol creates a global label with name \"GND\" , ground"
-			(at 106.68 109.22 0)
+			(at 106.68 111.76 0)
 			(effects
 				(font
@@
 			)
 		)
-		(property "Footprint" ""
+		(property "Footprint" "Capacitor_SMD:CP_Elec_10x10"
 			(at 74.6252 85.09 0)
 			(effects

Commit message: layoutig
Parts:
- C407, C408: footprint Capacitor_SMD:CP_Elec_10x10 -> Capacitor_SMD:CP_Elec_8x10.5
Changed lines of the file:
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@@
 			)
 		)
-		(property "Footprint" "Capacitor_SMD:CP_Elec_10x10"
+		(property "Footprint" "Capacitor_SMD:CP_Elec_8x10.5"
 			(at 74.6252 102.87 0)
 			(effects
@@
 			)
 		)
-		(property "Footprint" "Capacitor_SMD:CP_Elec_10x10"
+		(property "Footprint" "Capacitor_SMD:CP_Elec_8x10.5"
 			(at 74.6252 85.09 0)
 			(effects
