File: base-module.kicad_pcb (KiCad board)
At the start: 4 copper layers, 100 x 100 mm, 169 parts, among them J200 09031967921, J3 Programming header, J400 Conn_01x06_Socket, J401 Conn_01x06_Socket, J402 Conn_01x06_Socket, J403 Conn_01x06_Socket, J404 Conn_01x06_Socket, J405 XT60, Q700 MMST3904, U100 W25Q128, U300 TPS563200, U301 TPS563200, U302 CH334P, U400 STM32H563VGTx, U402 TPD2E2U06DCK, U403 DRV8844PWPR, U407 DRV8844PWPR, U500 TJA1044GTK_3Z, U600 TJA1044GTK_3Z, U700 STM32F103CBTx, X300 Q13FC1350000400, Y400 ASE-xxxMHz, Y700 8 MHz, Y900 12Mhz

Commit message: layout go brrr
Parts:
- removed LED406, LED408 (x2): FixLed307, FixLed307:FixLed307
- added C407: 47uF, Capacitor_SMD:CP_Elec_10x10, F.Cu at (87.2, 94.7)
- added C408: 47uF, Capacitor_SMD:CP_Elec_10x10, F.Cu at (110.9, 94.7)
- added C414: 47uF, Capacitor_SMD:CP_Elec_10x10, F.Cu at (72.9, 94.7)
- added C430: 47uF, Capacitor_SMD:CP_Elec_10x10, F.Cu at (49.2, 94.7)
- added C433: 100nF, PCM_JLCPCB:C_0402, F.Cu at (159.5, 106.9)
- added C435: 100nF, PCM_JLCPCB:C_0402, F.Cu at (64.1, 111.9)
- added C436: 100nF, PCM_JLCPCB:C_0402, F.Cu at (196.0, 107.7)
- added C437: 100nF, PCM_JLCPCB:C_0402, F.Cu at (174.4, 107.1)
- added C438: 100nF, PCM_JLCPCB:C_0402, F.Cu at (52.6, 111.9)
- added C439: 100nF, PCM_JLCPCB:C_0402, F.Cu at (224.7, 137.7)
- added C440: 100nF, PCM_JLCPCB:C_0402, F.Cu at (217.2, 136.9)
- added C441: 10nF, PCM_JLCPCB:C_0402, F.Cu at (156.0, 107.4)
- added C442: 10nF, PCM_JLCPCB:C_0402, F.Cu at (60.6, 112.4)
- added C443: 10nF, PCM_JLCPCB:C_0402, F.Cu at (192.5, 107.2)
- added C444: 10nF, PCM_JLCPCB:C_0402, F.Cu at (170.9, 107.6)
- added C445: 10nF, PCM_JLCPCB:C_0402, F.Cu at (49.0, 111.4)
- added C446: 10nF, PCM_JLCPCB:C_0402, F.Cu at (154.1, 99.1)
- added C447: 10nF, PCM_JLCPCB:C_0402, F.Cu at (56.7, 104.1)
- added C448: 10nF, PCM_JLCPCB:C_0402, F.Cu at (188.6, 99.9)
- added C449: 10nF, PCM_JLCPCB:C_0402, F.Cu at (169.0, 99.3)
- added C450: 10nF, PCM_JLCPCB:C_0402, F.Cu at (46.9, 104.0)
- added LED401: FixLed307, FixLed307:FixLed307, F.Cu at (104.6, 80.7)
- added LED403: FixLed307, FixLed307:FixLed307, F.Cu at (133.4, 67.9)
- added Q400: AO3400A, PCM_JLCPCB:Q_SOT-23, F.Cu at (153.0, 110.2)
- added Q401: AO3400A, PCM_JLCPCB:Q_SOT-23, F.Cu at (65.1, 108.8)
- added Q402: AO3401A, PCM_JLCPCB:Q_SOT-23, F.Cu at (156.7, 110.2)
- added Q403: AO3401A, PCM_JLCPCB:Q_SOT-23, F.Cu at (152.9, 101.7)
- added Q404: AO3400A, PCM_JLCPCB:Q_SOT-23, F.Cu at (189.5, 110.9)
- added Q405: AO3400A, PCM_JLCPCB:Q_SOT-23, F.Cu at (167.9, 110.3)
- added Q406: AO3401A, PCM_JLCPCB:Q_SOT-23, F.Cu at (61.4, 115.1)
- added Q407: AO3401A, PCM_JLCPCB:Q_SOT-23, F.Cu at (57.6, 106.6)
- added Q408: AO3400A, PCM_JLCPCB:Q_SOT-23, F.Cu at (45.8, 115.1)
- added Q410: AO3401A, PCM_JLCPCB:Q_SOT-23, F.Cu at (193.2, 110.9)
- added Q411: AO3401A, PCM_JLCPCB:Q_SOT-23, F.Cu at (189.4, 102.4)
- added Q414: AO3401A, PCM_JLCPCB:Q_SOT-23, F.Cu at (171.6, 110.3)
- added Q415: AO3401A, PCM_JLCPCB:Q_SOT-23, F.Cu at (167.8, 101.8)
- added Q418: AO3401A, PCM_JLCPCB:Q_SOT-23, F.Cu at (49.6, 115.1)
- added Q419: AO3401A, PCM_JLCPCB:Q_SOT-23, F.Cu at (45.8, 106.6)
- added Q420: AO3401A, PCM_JLCPCB:Q_SOT-23, F.Cu at (153.0, 105.9)
- added Q421: AO3401A, PCM_JLCPCB:Q_SOT-23, F.Cu at (57.6, 110.9)
- added Q422: AO3401A, PCM_JLCPCB:Q_SOT-23, F.Cu at (189.5, 106.7)
- added Q423: AO3401A, PCM_JLCPCB:Q_SOT-23, F.Cu at (167.9, 106.1)
- added Q424: AO3401A, PCM_JLCPCB:Q_SOT-23, F.Cu at (45.8, 110.8)
- added Q425: AO3401A, PCM_JLCPCB:Q_SOT-23, F.Cu at (156.8, 103.8)
- added Q426: AO3401A, PCM_JLCPCB:Q_SOT-23, F.Cu at (61.4, 108.8)
- added Q427: AO3401A, PCM_JLCPCB:Q_SOT-23, F.Cu at (193.3, 104.6)
- added Q428: AO3401A, PCM_JLCPCB:Q_SOT-23, F.Cu at (171.7, 104.0)
- added Q429: AO3401A, PCM_JLCPCB:Q_SOT-23, F.Cu at (49.6, 108.7)
- added Q430: AO3400A, PCM_JLCPCB:Q_SOT-23, F.Cu at (160.5, 103.8)
- added Q431: AO3400A, PCM_JLCPCB:Q_SOT-23, F.Cu at (57.6, 115.1)
- added Q432: AO3400A, PCM_JLCPCB:Q_SOT-23, F.Cu at (197.0, 104.6)
- added Q433: AO3400A, PCM_JLCPCB:Q_SOT-23, F.Cu at (175.4, 104.0)
- added Q434: AO3400A, PCM_JLCPCB:Q_SOT-23, F.Cu at (53.3, 108.7)
- added R407: 1kΩ, PCM_JLCPCB:R_0402, F.Cu at (158.5, 106.9)
- added R414: 0Ω, PCM_JLCPCB:R_0805, F.Cu at (156.8, 100.6)
- added R415: 0Ω, PCM_JLCPCB:R_0805, F.Cu at (160.5, 100.6)
- added R416: 220Ω, PCM_JLCPCB:R_0402, F.Cu at (219.0, 136.7)
- added R418: 1kΩ, PCM_JLCPCB:R_0402, F.Cu at (65.1, 111.9)
- added R419: 10kΩ, PCM_JLCPCB:R_0402, F.Cu at (60.6, 111.4)
- added R420: 10kΩ, PCM_JLCPCB:R_0402, F.Cu at (62.1, 111.9)
- added R421: 0Ω, PCM_JLCPCB:R_0805, F.Cu at (61.4, 105.6)
- added R422: 0Ω, PCM_JLCPCB:R_0805, F.Cu at (65.1, 105.6)
- added R423: 220Ω, PCM_JLCPCB:R_0402, F.Cu at (204.8, 136.9)
- added R424: 1kΩ, PCM_JLCPCB:R_0402, F.Cu at (195.0, 107.7)
- added R425: 1kΩ, PCM_JLCPCB:R_0402, F.Cu at (197.0, 107.7)
- added R426: 10kΩ, PCM_JLCPCB:R_0402, F.Cu at (192.5, 108.2)
- added R427: 10kΩ, PCM_JLCPCB:R_0402, F.Cu at (194.0, 107.7)
- added R428: 0Ω, PCM_JLCPCB:R_0805, F.Cu at (193.3, 101.4)
- added R429: 0Ω, PCM_JLCPCB:R_0805, F.Cu at (197.0, 101.4)
- added R430: 220Ω, PCM_JLCPCB:R_0402, F.Cu at (207.1, 145.7)
- added R431: 1kΩ, PCM_JLCPCB:R_0402, F.Cu at (173.4, 107.1)
- added R432: 1kΩ, PCM_JLCPCB:R_0402, F.Cu at (175.4, 107.1)
- added R433: 10kΩ, PCM_JLCPCB:R_0402, F.Cu at (170.9, 106.6)
- added R434: 10kΩ, PCM_JLCPCB:R_0402, F.Cu at (172.4, 107.1)
- added R435: 0Ω, PCM_JLCPCB:R_0805, F.Cu at (171.7, 100.8)
- added R436: 0Ω, PCM_JLCPCB:R_0805, F.Cu at (175.4, 100.8)
- added R437: 220Ω, PCM_JLCPCB:R_0402, F.Cu at (72.4, 81.0)
- added R438: 1kΩ, PCM_JLCPCB:R_0402, F.Cu at (51.6, 111.9)
- added R439: 1kΩ, PCM_JLCPCB:R_0402, F.Cu at (53.6, 111.9)
- added R440: 10kΩ, PCM_JLCPCB:R_0402, F.Cu at (49.0, 112.4)
- added R441: 10kΩ, PCM_JLCPCB:R_0402, F.Cu at (50.5, 111.9)
- added R442: 0Ω, PCM_JLCPCB:R_0805, F.Cu at (49.6, 105.5)
- added R443: 0Ω, PCM_JLCPCB:R_0805, F.Cu at (53.3, 105.5)
- added R444: 10kΩ, PCM_JLCPCB:R_0402, F.Cu at (215.3, 136.9)
- added R445: 10kΩ, PCM_JLCPCB:R_0402, F.Cu at (213.5, 136.9)
- added R446: 10kΩ, PCM_JLCPCB:R_0402, F.Cu at (211.6, 136.9)
- added R447: 10kΩ, PCM_JLCPCB:R_0402, F.Cu at (209.8, 136.9)
- added R448: 10kΩ, PCM_JLCPCB:R_0402, F.Cu at (207.9, 136.9)
- added R449: 10kΩ, PCM_JLCPCB:R_0402, F.Cu at (206.1, 136.9)
- added R450: 10kΩ, PCM_JLCPCB:R_0402, F.Cu at (224.7, 139.5)
- added R451: 10kΩ, PCM_JLCPCB:R_0402, F.Cu at (224.7, 141.4)
- added R452: 10kΩ, PCM_JLCPCB:R_0402, F.Cu at (224.7, 143.2)
- added R453: 10kΩ, PCM_JLCPCB:R_0402, F.Cu at (152.1, 99.1)
- added R454: 10kΩ, PCM_JLCPCB:R_0402, F.Cu at (224.7, 145.1)
- added R455: 10kΩ, PCM_JLCPCB:R_0402, F.Cu at (224.7, 146.9)
- added R456: 10kΩ, PCM_JLCPCB:R_0402, F.Cu at (224.7, 148.8)
- added R457: 10kΩ, PCM_JLCPCB:R_0402, F.Cu at (58.7, 104.1)
- added R458: 10kΩ, PCM_JLCPCB:R_0402, F.Cu at (190.6, 99.9)
- added R459: 10kΩ, PCM_JLCPCB:R_0402, F.Cu at (167.0, 99.3)
- added R460: 10kΩ, PCM_JLCPCB:R_0402, F.Cu at (44.9, 104.0)
- added R461: 10kΩ, PCM_JLCPCB:R_0402, F.Cu at (161.5, 106.9)
- added R462: 10kΩ, PCM_JLCPCB:R_0402, F.Cu at (66.1, 111.9)
- added R463: 10kΩ, PCM_JLCPCB:R_0402, F.Cu at (198.0, 107.7)
- added R464: 10kΩ, PCM_JLCPCB:R_0402, F.Cu at (176.4, 107.1)
- added R465: 10kΩ, PCM_JLCPCB:R_0402, F.Cu at (54.6, 111.9)
- added U401: SN74LVC1G19DBVR, Package_TO_SOT_SMD:SOT-23-6, F.Cu at (160.5, 110.2)
- added U404: SN74LVC1G19DBVR, Package_TO_SOT_SMD:SOT-23-6, F.Cu at (65.2, 115.1)
- added U405: SN74LVC1G19DBVR, Package_TO_SOT_SMD:SOT-23-6, F.Cu at (197.0, 110.9)
- added U406: SN74LVC1G19DBVR, Package_TO_SOT_SMD:SOT-23-6, F.Cu at (175.4, 110.3)
- added U408: TCA9535DBR, Package_SO:SSOP-24_5.3x8.2mm_P0.65mm, F.Cu at (213.1, 143.6)
- added U409: TCA9535DBR, Package_SO:SSOP-24_5.3x8.2mm_P0.65mm, F.Cu at (231.4, 141.8)
- added U410: SN74LVC1G19DBVR, Package_TO_SOT_SMD:SOT-23-6, F.Cu at (53.5, 115.1)
- R408, R417: value 220Ω -> 1kΩ
- R409, R413: value 220Ω -> 10kΩ
- moved R409 87.3 mm to (156.0, 106.4), turned to 180 degrees
- moved R408 78.4 mm to (160.5, 106.9)
- moved R413 62.6 mm to (157.5, 106.9)
- moved R417 58.4 mm to (63.1, 111.9)
- moved C409 41.1 mm to (106.0, 88.4), turned to -90 degrees
- moved C413 39.3 mm to (104.2, 92.4), turned to 180 degrees
- moved C411 30.2 mm to (92.7, 88.7), turned to -90 degrees
- moved U403 21.0 mm to (98.0, 92.2)
- moved C417 20.9 mm to (104.3, 90.0), turned to 90 degrees
- moved C419 19.7 mm to (93.7, 97.7), turned to -90 degrees
- moved C431 19.0 mm to (54.7, 88.7), turned to -90 degrees
- moved J401 14.2 mm to (64.7, 63.4)
- moved J400 14.0 mm to (50.6, 63.4)
- moved U407 13.4 mm to (59.9, 92.2)
- moved C412 13.3 mm to (66.2, 92.5), turned to 180 degrees
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Connections:
- net /Hbridge1-2/EN1 renamed /Hbridge1-2/BRIDGE.EN1
- net /Hbridge1-2/EN2 renamed /Hbridge1-2/BRIDGE.EN2
- net /Hbridge1-2/EN3 renamed /Hbridge1-2/BRIDGE.EN3
- net /Hbridge1-2/EN4 renamed /Hbridge1-2/BRIDGE.EN4
- net /Hbridge1-2/IN1 renamed /Hbridge1-2/BRIDGE.IN1
- net /Hbridge1-2/IN2 renamed /Hbridge1-2/BRIDGE.IN2
- net /Hbridge1-2/IN3 renamed /Hbridge1-2/BRIDGE.IN3
- net /Hbridge1-2/IN4 renamed /Hbridge1-2/BRIDGE.IN4
- net /Hbridge1-2/NFAULT1 renamed /Hbridge1-2/BRIDGE.NFAULT
- net /Hbridge1-2/NRST1 renamed /Hbridge1-2/BRIDGE.NRST
- net /Hbridge1-2/NSLEEP1 renamed /Hbridge1-2/BRIDGE.NSLEEP
- net /Hbridge3-4/EN1 renamed /Hbridge3-4/BRIDGE.EN1
- net /Hbridge3-4/EN2 renamed /Hbridge3-4/BRIDGE.EN2
- net /Hbridge3-4/EN3 renamed /Hbridge3-4/BRIDGE.EN3
- net /Hbridge3-4/EN4 renamed /Hbridge3-4/BRIDGE.EN4
- net /Hbridge3-4/IN1 renamed /Hbridge3-4/BRIDGE.IN1
- net /Hbridge3-4/IN2 renamed /Hbridge3-4/BRIDGE.IN2
- net /Hbridge3-4/IN3 renamed /Hbridge3-4/BRIDGE.IN3
- net /Hbridge3-4/IN4 renamed /Hbridge3-4/BRIDGE.IN4
- net /Hbridge3-4/NFAULT1 renamed /Hbridge3-4/BRIDGE.NFAULT
- net /Hbridge3-4/NRST1 renamed /Hbridge3-4/BRIDGE.NRST
- net /Hbridge3-4/NSLEEP1 renamed /Hbridge3-4/BRIDGE.NSLEEP
- J400 pad 1: /GPIO_Conn2/GPIO.LV+ -> /GPIO_Conn5/GPIO.LV+
- J400 pad 2: /GPIO_Conn2/GPIO.LV- -> GND
- J400 pad 3: /GPIO_Conn2/GPIO.Bridge+ -> /GPIO_Conn5/GPIO.Bridge+
- J400 pad 4: /GPIO_Conn2/GPIO.Bridge- -> /GPIO_Conn5/GPIO.Bridge-
- J400 pad 5: /GPIO_Conn2/GPIO.GPIO2 -> /GPIO_Conn5/GPIO.GPIO2
- J400 pad 6: /GPIO_Conn2/GPIO.GPIO1 -> /GPIO_Conn5/GPIO.GPIO1
- J401 pad 2: /GPIO_Conn1/GPIO.LV- -> GND
- J402 pad 1: /GPIO_Conn3/GPIO.LV+ -> /GPIO_Conn2/GPIO.LV+
- J402 pad 2: /GPIO_Conn3/GPIO.LV- -> GND
- J402 pad 3: /GPIO_Conn3/GPIO.Bridge+ -> /GPIO_Conn2/GPIO.Bridge+
- J402 pad 4: /GPIO_Conn3/GPIO.Bridge- -> /GPIO_Conn2/GPIO.Bridge-
- J402 pad 5: /GPIO_Conn3/GPIO.GPIO2 -> /GPIO_Conn2/GPIO.GPIO2
- J402 pad 6: /GPIO_Conn3/GPIO.GPIO1 -> /GPIO_Conn2/GPIO.GPIO1
- J403 pad 1: /GPIO_Conn4/GPIO.LV+ -> /GPIO_Conn3/GPIO.LV+
- J403 pad 2: /GPIO_Conn4/GPIO.LV- -> GND
- J403 pad 3: /GPIO_Conn4/GPIO.Bridge+ -> /GPIO_Conn3/GPIO.Bridge+
- J403 pad 4: /GPIO_Conn4/GPIO.Bridge- -> /GPIO_Conn3/GPIO.Bridge-
- J403 pad 5: /GPIO_Conn4/GPIO.GPIO2 -> /GPIO_Conn3/GPIO.GPIO2
- J403 pad 6: /GPIO_Conn4/GPIO.GPIO1 -> /GPIO_Conn3/GPIO.GPIO1
- J404 pad 1: /GPIO_Conn5/GPIO.LV+ -> /GPIO_Conn4/GPIO.LV+
- J404 pad 2: /GPIO_Conn5/GPIO.LV- -> GND
- J404 pad 3: /GPIO_Conn5/GPIO.Bridge+ -> /GPIO_Conn4/GPIO.Bridge+
- J404 pad 4: /GPIO_Conn5/GPIO.Bridge- -> /GPIO_Conn4/GPIO.Bridge-
- J404 pad 5: /GPIO_Conn5/GPIO.GPIO2 -> /GPIO_Conn4/GPIO.GPIO2
- J404 pad 6: /GPIO_Conn5/GPIO.GPIO1 -> /GPIO_Conn4/GPIO.GPIO1
- R400 pad 1: /GPIO_Conn1/LED -> /GPIO_Conn5/GPIO.LED
- R408 pad 1: /GPIO_Conn2/LED -> Net-(U401-Y1)
- R408 pad 2: Net-(LED402-Pad1) -> Net-(Q400-G)
- R409 pad 1: /GPIO_Conn3/LED -> Net-(Q402-G)
- R409 pad 2: Net-(LED404-Pad1) -> Net-(Q402-S)
- R413 pad 1: /GPIO_Conn4/LED -> Net-(U401-Y0)
- R413 pad 2: Net-(LED406-Pad1) -> GND
- R417 pad 1: /GPIO_Conn5/LED -> Net-(U404-Y0)
Routing:
- net Net-(Q400-G): track 0.00 -> 26.9 mm, vias 0 -> 4
- net Net-(Q407-S): track 0.00 -> 26.1 mm
- net Net-(Q400-D): track 0.00 -> 25.5 mm
- net Net-(Q402-G): track 0.00 -> 21.4 mm
- net Net-(Q408-G): track 0.00 -> 14.2 mm, vias 0 -> 2
- net Net-(Q419-S): track 0.00 -> 13.1 mm
- net Net-(Q411-S): track 0.00 -> 13.1 mm
- net Net-(Q403-S): track 0.00 -> 13.1 mm
- net Net-(Q405-G): track 0.00 -> 11.5 mm, vias 0 -> 2
- net Net-(Q404-G): track 0.00 -> 11.5 mm, vias 0 -> 2
- net Net-(Q404-D): track 0.00 -> 11.3 mm
- net (no net): track 11.0 -> 0.00 mm, vias 3 -> 0
- net Net-(Q418-G): track 0.00 -> 10.7 mm
- net Net-(Q410-G): track 0.00 -> 10.7 mm
- net Net-(Q414-G): track 0.00 -> 10.7 mm
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- added copper zone on F.Cu, net /GPIO_Conn1/GPIO.Bridge+
- added copper zone on F.Cu, net /GPIO_Conn1/GPIO.Bridge-
- added copper zone on F.Cu, net /GPIO_Conn2/GPIO.Bridge+
- added copper zone on F.Cu, net /GPIO_Conn2/GPIO.Bridge-
- added copper zone on F.Cu, net /Hbridge1-2/VM

Commit message: layouting
Parts:
- moved R416 133.4 mm to (89.8, 103.5), turned to 90 degrees
- moved U409 131.1 mm to (109.9, 92.5), turned to 90 degrees
- moved C440 130.7 mm to (91.2, 102.0), turned to 180 degrees
- moved U408 128.4 mm to (89.3, 109.5)
- moved R444 128.0 mm to (91.8, 103.5)
- moved R445 125.2 mm to (92.8, 103.5)
- moved R430 125.1 mm to (85.7, 115.4), turned to -90 degrees
- moved C439 125.0 mm to (105.8, 99.2), turned to 90 degrees
- moved R450 123.8 mm to (107.6, 99.2), turned to 90 degrees
- moved R447 123.6 mm to (90.8, 103.5), turned to 90 degrees
- moved R451 122.7 mm to (109.5, 99.2), turned to 90 degrees
- moved R446 122.5 mm to (91.0, 115.5), turned to 90 degrees
- moved R423 121.6 mm to (87.8, 103.6)
- moved R452 121.6 mm to (111.3, 99.2), turned to 90 degrees
- moved R454 120.6 mm to (113.2, 99.2), turned to 90 degrees
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Routing:
- net Net-(Q431-G): track 0.00 -> 17.3 mm, vias 0 -> 2
- net Net-(Q400-G): track 26.9 -> 18.3 mm, vias 4 -> 2
- net Net-(Q405-G): track 11.5 -> 18.4 mm
- net GND: track 110.6 -> 116.2 mm, vias 92 -> 94
- net Net-(Q404-G): track 11.5 -> 16.8 mm
- net Net-(Q408-D): track 8.10 -> 11.9 mm
- net Net-(Q408-G): track 14.2 -> 16.9 mm
- net Net-(Q401-G): track 0.00 -> 2.59 mm
- net Net-(Q430-G): track 5.12 -> 2.56 mm
- net Net-(U406-Y1): track 2.60 -> 1.00 mm

Commit message: layoutig
Parts:
- added C451: 47uF, Capacitor_SMD:CP_Elec_8x10.5, F.Cu at (128.8, 85.0)
- added C452: 47uF, Capacitor_SMD:CP_Elec_8x10.5, F.Cu at (128.8, 95.0)
- C407, C408, C414, C430: footprint Capacitor_SMD:CP_Elec_10x10 -> Capacitor_SMD:CP_Elec_8x10.5
- moved C414 79.7 mm to (111.2, 80.3), turned to 90 degrees
- moved R456 69.0 mm to (48.7, 89.0), turned to 180 degrees
- moved R455 68.9 mm to (46.2, 100.9), turned to 180 degrees
- moved R452 65.2 mm to (46.2, 101.8), turned to 0 degrees
- moved R454 65.2 mm to (48.7, 90.0), turned to 0 degrees
- moved R451 61.4 mm to (48.1, 100.9), turned to 0 degrees
- moved C439 60.4 mm to (46.2, 89.5)
- moved U409 60.2 mm to (49.7, 95.4)
- moved R450 59.6 mm to (48.1, 101.8), turned to 180 degrees
- moved C431 55.7 mm to (107.0, 90.2)
- moved C409 53.4 mm to (118.3, 91.1), turned to -90 degrees
- moved C408 52.9 mm to (82.6, 80.3), turned to 90 degrees
- moved Q408 52.6 mm to (98.4, 99.1), turned to 180 degrees
- moved C413 51.5 mm to (116.5, 95.2), turned to 180 degrees
- moved C417 51.2 mm to (116.6, 92.8), turned to 90 degrees
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Routing:
- net /GPIO_Conn5/GPIO.SEL: track 0.00 -> 46.0 mm, vias 0 -> 2
- net /GPIO_Conn5/GPIO.EN: track 0.00 -> 43.6 mm, vias 0 -> 2
- net /GPIO_Conn1/GPIO.SEL: track 0.00 -> 30.1 mm, vias 0 -> 2
- net /GPIO_Conn1/GPIO.EN: track 0.00 -> 29.3 mm, vias 0 -> 2
- net /GPIO_Conn3/GPIO.EN: track 0.00 -> 27.1 mm, vias 0 -> 2
- net GND: track 116.2 -> 142.0 mm, vias 94 -> 117
- net /GPIO_Conn2/GPIO.SEL: track 0.00 -> 24.8 mm, vias 0 -> 2
- net /GPIO_Conn3/GPIO.SEL: track 0.00 -> 24.8 mm, vias 0 -> 2
- net /GPIO_Conn2/GPIO.EN: track 0.00 -> 21.5 mm, vias 0 -> 2
- net Net-(Q401-G): track 2.59 -> 18.0 mm, vias 0 -> 2
- net Net-(Q431-G): track 17.3 -> 2.66 mm, vias 2 -> 0
- net +12V: track 0.00 -> 13.3 mm, vias 0 -> 9
- net Net-(Q402-G): track 21.4 -> 10.7 mm
- net Net-(Q406-G): track 0.00 -> 10.7 mm
- net +5V: track 38.2 -> 46.4 mm, vias 10 -> 14
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- added copper zone on F.Cu, net /GPIO_Conn1/GPIO.LV+
- added copper zone on F.Cu, net /GPIO_Conn2/GPIO.LV+
- added copper zone on F.Cu, net /GPIO_Conn3/GPIO.Bridge+
- added copper zone on F.Cu, net /GPIO_Conn3/GPIO.Bridge-
- added copper zone on F.Cu, net /GPIO_Conn3/GPIO.LV+
- added copper zone on F.Cu, net /GPIO_Conn4/GPIO.Bridge+
- added copper zone on F.Cu, net /GPIO_Conn4/GPIO.Bridge-
- added copper zone on F.Cu, net /GPIO_Conn4/GPIO.LV+
- added copper zone on F.Cu, net /GPIO_Conn5/GPIO.LV+
- removed copper zone on F.Cu, net /Hbridge1-2/VM
Other:
- board text added: "-"
