File: base-module.kicad_pcb (KiCad board)
At the start: 4 copper layers, 100 x 100 mm, 280 parts, among them J200 09031967921, J3 Programming header, J400 Conn_01x06_Socket, J401 Conn_01x06_Socket, J402 Conn_01x06_Socket, J403 Conn_01x06_Socket, J404 Conn_01x06_Socket, J405 XT60, Q400 AO3400A, Q401 AO3400A, Q402 AO3401A, Q403 AO3401A, Q404 AO3400A, Q405 AO3400A, Q406 AO3401A, Q407 AO3401A, Q408 AO3400A, Q410 AO3401A, Q411 AO3401A, Q414 AO3401A, Q415 AO3401A, Q418 AO3401A, Q419 AO3401A, Q420 AO3401A, Q421 AO3401A, Q422 AO3401A, Q423 AO3401A, Q424 AO3401A, Q425 AO3401A, Q426 AO3401A, Q427 AO3401A, Q428 AO3401A, Q429 AO3401A, Q430 AO3400A, Q431 AO3400A, Q432 AO3400A, Q433 AO3400A, Q434 AO3400A, Q700 MMST3904, U100 W25Q128, U300 TPS563200, U301 TPS563200, U302 CH334P, U400 STM32H563VGTx, U401 SN74LVC1G19DBVR, U402 TPD2E2U06DCK, U403 DRV8844PWPR, U404 SN74LVC1G19DBVR, U405 SN74LVC1G19DBVR, U406 SN74LVC1G19DBVR, U407 DRV8844PWPR, U408 TCA9535DBR, U409 TCA9535DBR, U410 SN74LVC1G19DBVR, U500 TJA1044GTK_3Z, U600 TJA1044GTK_3Z, U700 STM32F103CBTx, X300 Q13FC1350000400, Y400 ASE-xxxMHz, Y700 8 MHz, Y900 12Mhz

Commit message: a
Parts:
- added C1300: 10uF, PCM_JLCPCB:C_0603, F.Cu at (81.2, 105.8)
- added C1301: 100nF, PCM_JLCPCB:C_0402, F.Cu at (82.1, 109.9)
- added C1302: 100nF, PCM_JLCPCB:C_0402, F.Cu at (79.2, 106.6)
- added H400: MountingHole, MountingHole:MountingHole_3.5mm, F.Cu at (80.2, 133.6)
- added H401: MountingHole, MountingHole:MountingHole_3.5mm, F.Cu at (59.9, 133.6)
- added H402: MountingHole, MountingHole:MountingHole_3.5mm, F.Cu at (59.9, 118.4)
- added H403: MountingHole, MountingHole:MountingHole_3.5mm, F.Cu at (80.2, 118.4)
- added J406: Adafruit garbage connector, Connector_Molex:Molex_KK-254_AE-6410-06A_1x06_P2.54mm_Vertical, F.Cu at (63.7, 108.4)
- added U1300: BMP280, Package_LGA:Bosch_LGA-8_2x2.5mm_P0.65mm_ClockwisePinNumbering, F.Cu at (81.2, 107.9)
- added kibuzzard-6807DF1D: G***, kibuzzard-6807DF1D, F.Cu at (70.3, 125.8)
- moved R430 33.9 mm to (116.8, 88.4), turned to 0 degrees
- moved R416 28.5 mm to (102.6, 85.2), turned to 0 degrees
- moved C448 27.5 mm to (94.9, 115.4), turned to 0 degrees
- moved Q404 26.5 mm to (94.0, 104.3), turned to -90 degrees
- moved Q411 24.4 mm to (94.0, 112.8), turned to -90 degrees
- moved Q422 24.0 mm to (94.0, 108.6), turned to -90 degrees
- moved R458 23.8 mm to (92.9, 115.4), turned to 180 degrees
- moved C435 21.1 mm to (52.5, 130.4)
- moved R462 21.1 mm to (54.5, 130.4)
- moved C442 21.1 mm to (49.0, 130.9)
- moved Q401 21.1 mm to (46.0, 133.6)
- moved Q421 21.1 mm to (46.0, 129.4)
- moved R417 21.1 mm to (51.5, 130.4)
- moved R418 21.1 mm to (53.5, 130.4)
- moved R419 21.1 mm to (49.0, 129.9)
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Connections:
- net /I2C-GPIO/GPIO.SCL renamed /Barometer/BAROMETR_I2C.SCL
- net /I2C-GPIO/GPIO.SDA renamed /Barometer/BAROMETR_I2C.SDA
Routing:
- net /GPIO_Conn4/GPIO.GPIO1: track 0.00 -> 105.5 mm, vias 0 -> 1
- net /GPIO_Conn4/GPIO.GPIO2: track 0.00 -> 103.3 mm, vias 0 -> 1
- net /GPIO_Conn3/GPIO.GPIO1: track 0.00 -> 98.4 mm, vias 0 -> 1
- net /GPIO_Conn3/GPIO.GPIO2: track 0.00 -> 95.4 mm, vias 0 -> 1
- net /MCU/USR_BUTTON: track 1.22 -> 75.2 mm, vias 1 -> 6
- net /GPIO_Conn2/GPIO.GPIO1: track 0.00 -> 71.8 mm, vias 0 -> 1
- net /Barometer/BAROMETR_I2C.SCL: track 0.00 -> 70.1 mm, vias 0 -> 3
- net /MCU/SWD.~{RST}: track 26.9 -> 96.9 mm, vias 3 -> 8
- net /GPIO_Conn1/GPIO.GPIO1: track 0.00 -> 69.6 mm, vias 0 -> 1
- net /GPIO_Conn2/GPIO.GPIO2: track 0.00 -> 68.0 mm, vias 0 -> 1
- net /Barometer/BAROMETR_I2C.SDA: track 0.00 -> 68.0 mm, vias 0 -> 1
- net /GPIO_Conn1/GPIO.GPIO2: track 0.00 -> 64.2 mm, vias 0 -> 1
- net /GPIO_Conn4/GPIO.SEL: track 0.00 -> 50.4 mm, vias 0 -> 2
- net /GPIO_Conn5/GPIO.LED: track 0.00 -> 47.2 mm, vias 0 -> 6
- net /GPIO_Conn4/GPIO.EN: track 0.00 -> 46.4 mm, vias 0 -> 2
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- added copper zone on B.Cu, net /GPIO_Conn1/GPIO.Bridge+
- added copper zone on B.Cu, net /GPIO_Conn1/GPIO.LV+
- added copper zone on B.Cu, net /GPIO_Conn2/GPIO.Bridge+
- added copper zone on B.Cu, net /GPIO_Conn2/GPIO.LV+
- added copper zone on B.Cu, net /GPIO_Conn3/GPIO.Bridge+
- added copper zone on B.Cu, net /GPIO_Conn3/GPIO.LV+
- added copper zone on B.Cu, net /GPIO_Conn4/GPIO.Bridge+
- added copper zone on F.Cu, net /Hbridge1-2/VM
Other:
- board text added: "DOUBLE THE PERFORMANCE"
- board text added: "GPIO"
- board text removed: "DESIGNED IN POLAND"
