File: GPIO_Conn.kicad_sch (KiCad schematic)
At the start: 3 parts, among them J401 Conn_01x06_Socket

Commit message: layout go brrr
Parts:
- added C433: 100nF, PCM_JLCPCB:C_0402, symbol PCM_JLCPCB-Capacitors:0402,100nF,(2)
- added C441, C446: 10nF, PCM_JLCPCB:C_0402, symbol PCM_JLCPCB-Capacitors:0402,10nF
- added Q400, Q430: AO3400A, PCM_JLCPCB:Q_SOT-23, symbol PCM_JLCPCB-Transistors:NMOS,AO3400A
- added Q402, Q403, Q420, Q425: AO3401A, PCM_JLCPCB:Q_SOT-23, symbol PCM_JLCPCB-Transistors:PMOS,AO3401A
- added R407, R408: 1kΩ, PCM_JLCPCB:R_0402, symbol PCM_JLCPCB-Resistors:0402,1kΩ
- added R409, R413, R453, R461: 10kΩ, PCM_JLCPCB:R_0402, symbol PCM_JLCPCB-Resistors:0402,10kΩ
- added R414, R415: 0Ω, PCM_JLCPCB:R_0805, symbol PCM_JLCPCB-Resistors:0805,0Ω
- added U401: SN74LVC1G19DBVR, Package_TO_SOT_SMD:SOT-23-6, symbol 1to2Decoder:SN74LVC1G19DBVR
- renumbered J401 to J400
Connections:
- net GPIO.LV- is gone; now on net GND: J400.2 (Pin_2)
- net GND: now also C433.2, Q400.2 (S), Q430.2 (S), R413.2, R461.2, U401.2 (GND)
- net GPIO.LV+: now also Q420.3 (D), Q425.2 (S), R414.2, R415.2
- net LED renamed GPIO.LED
- new net: C441.1, Q402.1 (G), Q425.1 (G), Q430.3 (D), R409.1
- new net: C441.2, Q402.2 (S), Q425.3 (D), R409.2
- new net: Q430.1 (G), R407.2
- new net: R407.1, R413.1, U401.6 (Y0)
- new net: R408.1, R461.1, U401.4 (Y1)
- new net: C446.1, Q400.3 (D), Q403.1 (G), Q420.1 (G), R453.1
- new net: C446.2, Q403.2 (S), Q420.2 (S), R453.2
- new net: Q400.1 (G), R408.2
- new net +12V: Q403.3 (D), R415.1
- new net +3V3: C433.1, U401.5 (VCC)
- new net +5V: Q402.3 (D), R414.1
- new net GPIO.EN: U401.3 (~{E})
- new net GPIO.SEL: U401.1 (A)
Other:
- moved on the sheet: J400, LED400A, LED400B, R400

Commit message: a
Changed lines of the file:
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@@
+	)
+	(junction
+		(at 193.04 29.21)
+		(diameter 0)
+		(color 0 0 0 0)
 	)
 	(junction
@@
 	)
 	(junction
-		(at 193.04 31.75)
-		(diameter 0)
-		(color 0 0 0 0)
-	)
-	(junction
 		(at 149.86 113.03)
 		(diameter 0)
@@
 	)
 	(junction
-		(at 193.04 96.52)
+		(at 205.74 69.85)
 		(diameter 0)
 		(color 0 0 0 0)
@@
 	)
 	(junction
+		(at 193.04 93.98)
+		(diameter 0)
+		(color 0 0 0 0)
+	)
+	(junction
 		(at 121.92 62.23)
 		(diameter 0)
@@
 	)
 	(junction
-		(at 205.74 66.04)
-		(diameter 0)
-		(color 0 0 0 0)
-	)
-	(junction
 		(at 153.67 55.88)
 		(diameter 0)
@@
 	)
 	(junction
-		(at 205.74 133.35)
+		(at 205.74 137.16)
 		(diameter 0)
 		(color 0 0 0 0)
@@
 	(wire
 		(pts
-			(xy 205.74 31.75) (xy 193.04 31.75)
+			(xy 205.74 29.21) (xy 193.04 29.21)
 		)
 		(stroke
@@
 	(wire
 		(pts
-			(xy 193.04 133.35) (xy 205.74 133.35)
+			(xy 193.04 137.16) (xy 205.74 137.16)
 		)
 		(stroke
@@
 	(wire
 		(pts
-			(xy 205.74 114.3) (xy 205.74 133.35)
+			(xy 193.04 69.85) (xy 193.04 66.04)
+		)
+		(stroke
+			(width 0)
+			(type default)
+		)
+	)
+	(wire
+		(pts
+			(xy 205.74 114.3) (xy 205.74 137.16)
+		)
+		(stroke
+			(width 0)
+			(type default)
+		)
+	)
+	(wire
+		(pts
+			(xy 205.74 53.34) (xy 205.74 69.85)
 		)
 		(stroke
@@
 	(wire
 		(pts
-			(xy 193.04 88.9) (xy 193.04 96.52)
+			(xy 193.04 88.9) (xy 193.04 93.98)
 		)
 		(stroke
@@
 	(wire
 		(pts
-			(xy 193.04 96.52) (xy 193.04 97.79)
-		)
-		(stroke
-			(width 0)
-			(type default)
-		)
-	)
-	(wire
-		(pts
 			(xy 107.95 62.23) (xy 121.92 62.23)
 		)
@@
 	(wire
 		(pts
-			(xy 193.04 24.13) (xy 193.04 31.75)
+			(xy 193.04 24.13) (xy 193.04 29.21)
 		)
 		(stroke
@@
 	(wire
 		(pts
-			(xy 193.04 66.04) (xy 205.74 66.04)
+			(xy 193.04 69.85) (xy 205.74 69.85)
 		)
 		(stroke
@@
 	(wire
 		(pts
-			(xy 205.74 66.04) (xy 219.71 66.04)
+			(xy 205.74 69.85) (xy 219.71 69.85)
 		)
 		(stroke
@@
 	(wire
 		(pts
-			(xy 193.04 130.81) (xy 193.04 133.35)
-		)
-		(stroke
-			(width 0)
-			(type default)
-		)
-	)
-	(wire
-		(pts
-			(xy 205.74 106.68) (xy 205.74 96.52)
+			(xy 193.04 130.81) (xy 193.04 137.16)
+		)
+		(stroke
+			(width 0)
+			(type default)
+		)
+	)
+	(wire
+		(pts
+			(xy 193.04 93.98) (xy 193.04 97.79)
+		)
+		(stroke
+			(width 0)
+			(type default)
+		)
+	)
+	(wire
+		(pts
+			(xy 205.74 106.68) (xy 205.74 93.98)
 		)
 		(stroke
@@
 	(wire
 		(pts
+			(xy 193.04 29.21) (xy 193.04 33.02)
+		)
+		(stroke
+			(width 0)
+			(type default)
+		)
+	)
+	(wire
+		(pts
 			(xy 149.86 86.36) (xy 149.86 113.03)
 		)
@@
 	(wire
 		(pts
-			(xy 205.74 133.35) (xy 219.71 133.35)
+			(xy 205.74 137.16) (xy 219.71 137.16)
 		)
 		(stroke
@@
 	(wire
 		(pts
-			(xy 205.74 31.75) (xy 205.74 45.72)
-		)
-		(stroke
-			(width 0)
-			(type default)
-		)
-	)
-	(wire
-		(pts
-			(xy 205.74 53.34) (xy 205.74 66.04)
+			(xy 205.74 29.21) (xy 205.74 45.72)
 		)
 		(stroke
@@
 	(wire
 		(pts
-			(xy 193.04 31.75) (xy 193.04 33.02)
-		)
-		(stroke
-			(width 0)
-			(type default)
-		)
-	)
-	(wire
-		(pts
 			(xy 149.86 124.46) (xy 149.86 125.73)
 		)
@@
 	(wire
 		(pts
-			(xy 219.71 66.04) (xy 219.71 92.71)
+			(xy 219.71 69.85) (xy 219.71 92.71)
 		)
 		(stroke
@@
 	(wire
 		(pts
-			(xy 205.74 96.52) (xy 193.04 96.52)
+			(xy 205.74 93.98) (xy 193.04 93.98)
 		)
 		(stroke
@@
 	(wire
 		(pts
-			(xy 219.71 92.71) (xy 219.71 133.35)
-		)
-		(stroke
+			(xy 219.71 92.71) (xy 219.71 137.16)
+		)
+		(stroke
