File: base-module.kicad_sch (KiCad schematic)
At the start: 1 part, among them J405 XT60

Commit message: layout go brrr
Other:
- removed sheet Power_Switch1
- removed sheet Power_Switch2
- removed sheet Power_Switch3
- removed sheet Power_Switch4
- sheet GPIO_Conn1 ports: added none; removed LED
- sheet GPIO_Conn2 ports: added none; removed LED
- sheet GPIO_Conn3 ports: added none; removed LED
- sheet GPIO_Conn4 ports: added none; removed LED
- sheet I2C-GPIO ports: added GPIO{I2C}; removed none
- sheet I2C_pwr_sel ports: added GPIO1{GPIO_CONN}, GPIO2{GPIO_CONN}, GPIO3{GPIO_CONN}, GPIO4{GPIO_CONN}, GPIO5{GPIO_CONN}, PWR_SEL{I2C}; removed none
- moved on the sheet: J405

Commit message: layoutig
Parts:
- added C451, C452: 47uF, Capacitor_SMD:CP_Elec_8x10.5, symbol Device:C_Polarized
Connections:
- net GND: now also C451.2, C452.2
- net Hbridge1-2/V_conn: now also C451.1, C452.1

Commit message: a
Other:
- added sheet Barometer (Barometer.kicad_sch)
- added sheet IMU (IMU.kicad_sch)
- moved on the sheet: C451, C452, J405
