File: mcu.kicad_sch (KiCad schematic)
At the start: 33 parts, among them U400 STM32H563VGTx, X300 Q13FC1350000400, Y400 ASE-xxxMHz

Commit message: layout go brrr
Connections:
- no-connect marks 56 -> 62
Other:
- moved on the sheet: BTN400A, C416, R405, R406

Commit message: a
Connections:
- net PC0: now reaches U400.15 (PC0)
- net PC1: now reaches U400.16 (PC1)
- net PC2: now reaches U400.17 (PC2)
- net PC3: now reaches U400.18 (PC3)
- net PA0: now reaches U400.23 (PA0)
- net PA1: now reaches U400.24 (PA1)
- net PA2: now reaches U400.25 (PA2)
- net PA3: now reaches U400.26 (PA3)
- net PA4: now reaches U400.29 (PA4)
- net PA5: now reaches U400.30 (PA5)
- net PA6: now reaches U400.31 (PA6)
- net PA7: now reaches U400.32 (PA7)
- net PC4: now reaches U400.33 (PC4)
- net PC5: now reaches U400.34 (PC5)
- net PE7: now reaches U400.38 (PE7)
- net PE8: now reaches U400.39 (PE8)
- net PE9: now reaches U400.40 (PE9)
- net PE10: now reaches U400.41 (PE10)
- net PE11: now reaches U400.42 (PE11)
- net PE12: now reaches U400.43 (PE12)
- net PE13: now reaches U400.44 (PE13)
- net PE14: now reaches U400.45 (PE14)
- net PE15: now reaches U400.46 (PE15)
- net PB14: now reaches U400.53 (PB14)
- net PB15: now reaches U400.54 (PB15)
- net PD8: now reaches U400.55 (PD8)
- net PD9: now reaches U400.56 (PD9)
- net PD10: now reaches U400.57 (PD10)
- net PD14: now reaches U400.61 (PD14)
- net PD15: now reaches U400.62 (PD15)
- net PC6: now reaches U400.63 (PC6)
- net PC7: now reaches U400.64 (PC7)
- net PC8: now reaches U400.65 (PC8)
- net PC9: now reaches U400.66 (PC9)
- net PA8: now reaches U400.67 (PA8)
- net PA9: now reaches U400.68 (PA9)
- net PA10: now reaches U400.69 (PA10)
- net PC13: now reaches U400.7 (PC13)
- net PC10: now reaches U400.78 (PC10)
- net PC11: now reaches U400.79 (PC11)
- net PC12: now reaches U400.80 (PC12)
- net PD2: now reaches U400.83 (PD2)
- net PD3: now reaches U400.84 (PD3)
- net PD4: now reaches U400.85 (PD4)
- net PD5: now reaches U400.86 (PD5)
- net PD6: now reaches U400.87 (PD6)
- net PD7: now reaches U400.88 (PD7)
- no-connect marks 62 -> 15
